File: hardware/VCAT-pedalsBoardPCB/pedalsBoard/PowerProtection.kicad_sch (KiCad schematic)
At the start: 18 parts, among them IC2 LM74502DDFR, Q2 PSMN012-100YS, Q3 PSMN012-100YS

Commit message: monday evening check
Parts:
- renumbered C32 to C48, C33 to C49, C34 to C50, C35 to C51, C36 to C52, C37 to C53, C38 to C54, D6 to D11, D7 to D12, IC2 to IC3, Q2 to Q4, Q3 to Q6, R11 to R24, R15 to R25, R16 to R26, R17 to R27, R18 to R28, R19 to R29
