File: hardware/VCAT-pedalsBoardPCB/pedalsBoard/pedalsBoard.kicad_sch (KiCad schematic)
At the start: 10 parts, among them J1 CAN_NANO_01x05, J2 CAN_DEBUG_NANO_01x04, J5 CAN_NANO_01x05, J6 Conn_02x04_Counter_Clockwise, J8 Conn_02x03_Counter_Clockwise

Commit message: implemented review suggestions and added bus
Other:
- sheet MCU ports: added {SENS_READINGS}; removed ACCPOT_1, ACCPOT_2, B_SENS_1, B_SENS_2, B_SWCH_OUT
- sheet SensorLogic ports: added {SENS_RAW}, {SENS_READINGS}; removed ACCEL1_OUT, ACCEL2_OUT, ACCPOT_1, ACCPOT_2, B_SENS, B_SENSOUT1, B_SENSOUT2, B_SWCH_OUT, B_SWITCH
- note removed: "Sensor Inputs"
- note removed: "Sensor Outputs"
