File: hardware/VCAT-pedalsBoardPCB/pedalsBoard/pedalsBoard.kicad_sch (KiCad schematic)
At the start: 10 parts, among them J1 CAN_NANO_01x05, J2 CAN_DEBUG_NANO_01x04, J5 CAN_NANO_01x05, J6 Conn_02x04_Counter_Clockwise, J8 Conn_02x03_Counter_Clockwise

Commit message: addressed review, brake switch on slack
Parts:
- removed F12, F13: Fuse, MyParts:FUSC1709X80N, symbol Device:Fuse
- removed R15: 0, Resistor_SMD:R_0603_1608Metric_Pad0.98x0.95mm_HandSolder, symbol Device:R
- removed R6: 0, symbol Device:R
- added F2: Fuse, MyParts:FUSC1709X80N, symbol Device:Polyfuse
- added R1: 0, symbol Device:R
- F1: renamed from F11; symbol Device:Fuse -> Device:Polyfuse
- renumbered J6 to J1, J1 to J2, J5 to J3, J2 to J4, J8 to J5
Connections:
- net V_IN is gone; now on net +12V: J2.1 (12V), J3.1 (12V), J4.1 (12V)
- net +5V: now also F2.2
- net GND: now also R1.1
- net at J5.1 (Pin_1): now also J5.6 (Pin_6), F2.1
- net at J2.5 (SHIELD): now also J3.5 (SHIELD), R1.2
Other:
- sheet MCU ports: added 5V_USB; removed 5V
- sheet Power ports: added none; removed 12V
- sheet SensorLogic ports: added GNDA, VDDA; removed 5V
- note added: "Each Pot Max Draw: 11mA * 2 = 22mA 50 mA Fuse?"
- note added: "Shielding"
- note removed: "CAN"
- note removed: "CAN Connection to BUS"
- note removed: "Debug"
- note removed: "MCU and USB"
- note removed: "Power In"
- note removed: "Sensor Logic"
- moved on the sheet: J1, J2, J3, J4, J5
