File: hardware/VCAT-pedalsBoardPCB/pedalsBoard/pedalsBoard.kicad_sch (KiCad schematic)
At the start: 11 parts, among them J11 Conn_01x04, J2 CAN_NANO_01x05, J3 CAN_NANO_01x05, J5 Conn_02x03_Counter_Clockwise, J6 DEBUG_CAN, SW3 SW_CONN

Commit message: tweaked some power labels
Connections:
- net +12V: no longer J2.1 (12V), J3.1 (12V), J6.1 (12V)
- new net +12V_PP: J2.1 (12V), J3.1 (12V), J6.1 (12V)
Other:
- sheet Power ports: added +12V_PP; removed none
