File: hardware/VCAT-pedalsBoardPCB/pedalsBoard/48PinMCU.kicad_sch (KiCad schematic)
At the start: 34 parts, among them J1 SWD_Header, J2 SWD, SW1 Reset, SW2 SW_SPDT, U1 STM32G473CETx, Y1 Crystal

Commit message: monday evening check
Connections:
- net USB_DM renamed PA11
- net USB_DP renamed PA12
Changed lines of the file:
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@@
+		)
+	)
+	(hierarchical_label "PA11"
+		(shape bidirectional)
+		(at 121.92 64.77 0)
+		(effects
+			(font
+				(size 1.27 1.27)
+			)
+			(justify left)
 		)
 	)
@@
 		)
 	)
-	(hierarchical_label "USB_DM"
-		(shape bidirectional)
-		(at 121.92 64.77 0)
-		(effects
-			(font
-				(size 1.27 1.27)
-			)
-			(justify left)
-		)
-	)
-	(hierarchical_label "USB_DP"
+	(hierarchical_label "PB12"
+		(shape bidirectional)
+		(at 60.96 92.71 180)
+		(effects
+			(font
+				(size 1.27 1.27)
+			)
+			(justify right)
+		)
+	)
+	(hierarchical_label "PA12"
 		(shape bidirectional)
 		(at 121.92 67.31 0)
@@
 		)
 	)
-	(hierarchical_label "PB12"
-		(shape bidirectional)
-		(at 60.96 92.71 180)
-		(effects
-			(font
-				(size 1.27 1.27)
-			)
-			(justify right)
-		)
-	)

Commit message: meow
Parts:
- renumbered C1 to C20, C2 to C21, C3 to C26, C4 to C27, C5 to C28, C6 to C29, C7 to C30, C8 to C31, C9 to C32, C10 to C33, C11 to C34, C12 to C35, C13 to C36, C14 to C37, C15 to C38, D1 to D5, D2 to D6, D3 to D7, FB1 to FB3, FB2 to FB4, J1 to J3, J2 to J4, R1 to R12, R2 to R13, R3 to R19, R4 to R30, R5 to R31, R6 to R32, R7 to R33, R8 to R34, SW1 to SW3, SW2 to SW4, U1 to U2, Y1 to Y2

Commit message: addressed review, brake switch on slack
Parts:
- renumbered C37 to C12, C27 to C13, C29 to C14, C31 to C15, C33 to C16, C35 to C17, C36 to C18, C20 to C19, C21 to C20, C38 to C21, C26 to C22, C30 to C23, C32 to C24, C34 to C25, C28 to C26, D6 to D10, D7 to D11, D5 to D12, FB4 to FB1, FB3 to FB2, J3 to J7, J4 to J8, R13 to R19, R33 to R20, R34 to R21, R31 to R22, R32 to R23, R12 to R24, R19 to R25, R30 to R26, SW4 to SW1, SW3 to SW2, U2 to U4, Y2 to Y1
