File: hardware/VCAT-pedalsBoardPCB/pedalsBoard/48PinMCU.kicad_sch (KiCad schematic)
At the start: 34 parts, among them J7 SWD_Header, J8 SWD, SW1 SW_SPDT, SW2 Reset, U4 STM32G473CETx, Y1 Crystal

Commit message: hopefully final before layout
Other:
- moved on the sheet: C12, C14, C17, C19, C20, C21, C22, C23, C24, C25, C26, FB1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
