File: hardware/VCAT-pedalsBoardPCB/pedalsBoard/PP.kicad_sch (KiCad schematic)
At the start: 18 parts, among them IC3 LM74502DDFR, Q4 PSMN012-100YS, Q6 PSMN012-100YS

Commit message: addressed review, brake switch on slack
Parts:
- IC2: renamed from IC3; Manufacturer_Name Texas Instruments -> (none); Manufacturer_Part_Number LM74502DDFR -> (none); Mouser Part Number 595-LM74502DDFR -> (none); Mouser Price/Stock https://www.mouser.co.uk/ProductDetail/Texas-Instruments/LM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 -> (none)
- R34: renamed from R25; symbol Device:R_US -> Device:R; Mouser Part Number 594-MCT06030C3309FP5 -> (none)
- R35: renamed from R24; symbol Device:R_US -> Device:R
- R36: renamed from R26; symbol Device:R_US -> Device:R
- R37: renamed from R28; symbol Device:R_US -> Device:R
- R38: renamed from R27; symbol Device:R_US -> Device:R
- R39: renamed from R29; symbol Device:R_US -> Device:R
- renumbered C48 to C41, C52 to C42, C51 to C43, C50 to C44, C49 to C45, C53 to C46, C54 to C47, D11 to D14, D12 to D15, Q4 to Q1, Q6 to Q2
Other:
- note added: "Supp Battery Range: 10V-14.7V"
