File: hardware/VCAT-pedalsBoardPCB/pedalsBoard/Power_Mux.kicad_sch (KiCad schematic)
At the start: 6 parts, among them U1 TPS2117DRLR

Commit message: addressed review, brake switch on slack
Parts:
- renumbered C1 to C31, C2 to C32, C4 to C33, C3 to C34, R1 to R31, U1 to U5
Changed lines of the file:
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@@
 		(in_pos_files yes)
 		(dnp no)
-		(property "Reference" "C4"
+		(property "Reference" "C33"
 			(at 91.8972 57.2516 0)
 			(show_name no)
@@
 		(instances
 			(project "pedalsBoard"
-				(path "/423853f6-a5c6-4d97-9a9a-db6f143664c7/26d9f075-73a6-4044-b4f9-8fe225c47fcc/acc44d2c-6102-4029-853a-d596701ce5ec"
-					(reference "C4")
+				(path "/423853f6-a5c6-4d97-9a9a-db6f143664c7/26d9f075-73a6-4044-b4f9-8fe225c47fcc/0b4834e3-0a71-44a6-a6c4-c6d53fe5e39e"
+					(reference "C33")
 					(unit 1)
 				)
@@
 		(in_pos_files yes)
 		(dnp no)
-		(property "Reference" "R1"
+		(property "Reference" "R31"
 			(at 78.994 67.564 0)
 			(show_name no)
@@
 		(instances
 			(project "pedalsBoard"
-				(path "/423853f6-a5c6-4d97-9a9a-db6f143664c7/26d9f075-73a6-4044-b4f9-8fe225c47fcc/acc44d2c-6102-4029-853a-d596701ce5ec"
-					(reference "R1")
+				(path "/423853f6-a5c6-4d97-9a9a-db6f143664c7/26d9f075-73a6-4044-b4f9-8fe225c47fcc/0b4834e3-0a71-44a6-a6c4-c6d53fe5e39e"
+					(reference "R31")
 					(unit 1)
 				)
@@
 		(in_pos_files yes)
 		(dnp no)
-		(property "Reference" "C1"
+		(property "Reference" "C31"
 			(at 24.5872 44.5516 0)
 			(show_name no)
@@
 		(instances
 			(project "pedalsBoard"
-				(path "/423853f6-a5c6-4d97-9a9a-db6f143664c7/26d9f075-73a6-4044-b4f9-8fe225c47fcc/acc44d2c-6102-4029-853a-d596701ce5ec"
-					(reference "C1")
+				(path "/423853f6-a5c6-4d97-9a9a-db6f143664c7/26d9f075-73a6-4044-b4f9-8fe225c47fcc/0b4834e3-0a71-44a6-a6c4-c6d53fe5e39e"
+					(reference "C31")
 					(unit 1)
 				)
@@
 		(dnp no)
 		(fields_autoplaced yes)
-		(property "Reference" "U1"
+		(property "Reference" "U5"
 			(at 60.96 44.45 0)
 			(show_name no)
@@
 		(instances
 			(project "pedalsBoard"
-				(path "/423853f6-a5c6-4d97-9a9a-db6f143664c7/26d9f075-73a6-4044-b4f9-8fe225c47fcc/acc44d2c-6102-4029-853a-d596701ce5ec"
-					(reference "U1")
+				(path "/423853f6-a5c6-4d97-9a9a-db6f143664c7/26d9f075-73a6-4044-b4f9-8fe225c47fcc/0b4834e3-0a71-44a6-a6c4-c6d53fe5e39e"
+					(reference "U5")
 					(unit 1)
 				)
@@
 		(in_pos_files yes)
 		(dnp no)
-		(property "Reference" "C3"
+		(property "Reference" "C34"
 			(at 42.3672 67.4116 0)
 			(show_name no)
@@
 		(instances
 			(project "pedalsBoard"
-				(path "/423853f6-a5c6-4d97-9a9a-db6f143664c7/26d9f075-73a6-4044-b4f9-8fe225c47fcc/acc44d2c-6102-4029-853a-d596701ce5ec"
-					(reference "C3")
+				(path "/423853f6-a5c6-4d97-9a9a-db6f143664c7/26d9f075-73a6-4044-b4f9-8fe225c47fcc/0b4834e3-0a71-44a6-a6c4-c6d53fe5e39e"
+					(reference "C34")
 					(unit 1)
 				)
@@
 		(in_pos_files yes)
 		(dnp no)
-		(property "Reference" "C2"
+		(property "Reference" "C32"
 			(at 38.5572 44.5516 0)
 			(show_name no)
@@
 		(instances
 			(project "pedalsBoard"
-				(path "/423853f6-a5c6-4d97-9a9a-db6f143664c7/26d9f075-73a6-4044-b4f9-8fe225c47fcc/acc44d2c-6102-4029-853a-d596701ce5ec"
-					(reference "C2")
+				(path "/423853f6-a5c6-4d97-9a9a-db6f143664c7/26d9f075-73a6-4044-b4f9-8fe225c47fcc/0b4834e3-0a71-44a6-a6c4-c6d53fe5e39e"
+					(reference "C32")
 					(unit 1)
 				)
