File: hardware/VCAT-pedalsBoardPCB/pedalsBoard/12VBuck.kicad_sch (KiCad schematic)
At the start: 14 parts, among them U4 LMR51635XDDCR

Commit message: monday evening check
Parts:
- renumbered C24 to C40, C25 to C41, C26 to C42, C27 to C43, C28 to C44, C29 to C45, L1 to L2, R13 to R22, R14 to R23, TP1 to TP5, TP2 to TP6, TP3 to TP7, TP4 to TP8, U4 to U6

Commit message: test
Parts:
- removed TP6: CB, TestPoint:TestPoint_THTPad_D3.0mm_Drill1.5mm, symbol Connector:TestPoint
- removed TP7: FB, TestPoint:TestPoint_THTPad_D3.0mm_Drill1.5mm, symbol Connector:TestPoint
- removed TP8: SW, TestPoint:TestPoint_THTPad_D3.0mm_Drill1.5mm, symbol Connector:TestPoint
- R22, R23: footprint Resistor_SMD:R_0603_1608Metric -> Resistor_SMD:R_0603_1608Metric_Pad0.98x0.95mm_HandSolder

Commit message: addressed review, brake switch on slack
Parts:
- renumbered C42 to C35, C40 to C36, C41 to C37, C43 to C38, C44 to C39, C45 to C40, L2 to L1, R22 to R32, R23 to R33, TP5 to TP14
Changed lines of the file:
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@@
 		(dnp no)
 		(fields_autoplaced yes)
-		(property "Reference" "#FLG07"
+		(property "Reference" "#FLG09"
 			(at 149.86 79.375 0)
 			(hide yes)
@@
 		(instances
 			(project "pedalsBoard"
-				(path "/423853f6-a5c6-4d97-9a9a-db6f143664c7/26d9f075-73a6-4044-b4f9-8fe225c47fcc/201cb619-540d-483a-b529-2226b2b1f1d1"
-					(reference "#FLG07")
+				(path "/423853f6-a5c6-4d97-9a9a-db6f143664c7/26d9f075-73a6-4044-b4f9-8fe225c47fcc/521dc22e-9478-4c61-a4c9-c65800ada9dd"
+					(reference "#FLG09")
 					(unit 1)
 				)
@@
 		(dnp no)
 		(fields_autoplaced yes)
-		(property "Reference" "C40"
+		(property "Reference" "C36"
 			(at 96.52 85.0962 0)
 			(show_name no)
@@
 		(instances
 			(project "pedalsBoard"
-				(path "/423853f6-a5c6-4d97-9a9a-db6f143664c7/26d9f075-73a6-4044-b4f9-8fe225c47fcc/201cb619-540d-483a-b529-2226b2b1f1d1"
-					(reference "C40")
+				(path "/423853f6-a5c6-4d97-9a9a-db6f143664c7/26d9f075-73a6-4044-b4f9-8fe225c47fcc/521dc22e-9478-4c61-a4c9-c65800ada9dd"
+					(reference "C36")
 					(unit 1)
 				)
@@
 		(in_pos_files yes)
 		(dnp no)
-		(property "Reference" "TP5"
+		(property "Reference" "TP14"
 			(at 229.87 123.6979 0)
 			(hide yes)
@@
 		(instances
 			(project "pedalsBoard"
-				(path "/423853f6-a5c6-4d97-9a9a-db6f143664c7/26d9f075-73a6-4044-b4f9-8fe225c47fcc/201cb619-540d-483a-b529-2226b2b1f1d1"
-					(reference "TP5")
+				(path "/423853f6-a5c6-4d97-9a9a-db6f143664c7/26d9f075-73a6-4044-b4f9-8fe225c47fcc/521dc22e-9478-4c61-a4c9-c65800ada9dd"
+					(reference "TP14")
 					(unit 1)
 				)
@@
 		(in_pos_files yes)
 		(dnp no)
-		(property "Reference" "L2"
+		(property "Reference" "L1"
 			(at 161.29 87.884 90)
 			(show_name no)
@@
 		(instances
 			(project "pedalsBoard"
-				(path "/423853f6-a5c6-4d97-9a9a-db6f143664c7/26d9f075-73a6-4044-b4f9-8fe225c47fcc/201cb619-540d-483a-b529-2226b2b1f1d1"
-					(reference "L2")
+				(path "/423853f6-a5c6-4d97-9a9a-db6f143664c7/26d9f075-73a6-4044-b4f9-8fe225c47fcc/521dc22e-9478-4c61-a4c9-c65800ada9dd"
+					(reference "L1")
 					(unit 1)
 				)
@@
 		(dnp no)
 		(fields_autoplaced yes)
-		(property "Reference" "#FLG09"
+		(property "Reference" "#FLG011"
 			(at 179.07 84.455 0)
 			(hide yes)
@@
 		(instances
 			(project "pedalsBoard"
-				(path "/423853f6-a5c6-4d97-9a9a-db6f143664c7/26d9f075-73a6-4044-b4f9-8fe225c47fcc/201cb619-540d-483a-b529-2226b2b1f1d1"
-					(reference "#FLG09")
+				(path "/423853f6-a5c6-4d97-9a9a-db6f143664c7/26d9f075-73a6-4044-b4f9-8fe225c47fcc/521dc22e-9478-4c61-a4c9-c65800ada9dd"
+					(reference "#FLG011")
 					(unit 1)
 				)
@@
 		(dnp no)
 		(fields_autoplaced yes)
-		(property "Reference" "#FLG06"
+		(property "Reference" "#FLG08"
 			(at 88.9 79.375 0)
 			(hide yes)
@@
 		(instances
 			(project "pedalsBoard"
-				(path "/423853f6-a5c6-4d97-9a9a-db6f143664c7/26d9f075-73a6-4044-b4f9-8fe225c47fcc/201cb619-540d-483a-b529-2226b2b1f1d1"
-					(reference "#FLG06")
+				(path "/423853f6-a5c6-4d97-9a9a-db6f143664c7/26d9f075-73a6-4044-b4f9-8fe225c47fcc/521dc22e-9478-4c61-a4c9-c65800ada9dd"
+					(reference "#FLG08")
 					(unit 1)
 				)
@@
 		(in_pos_files yes)
 		(dnp no)
-		(property "Reference" "C43"
+		(property "Reference" "C38"
 			(at 164.084 93.98 0)
 			(show_name no)
@@
 		(instances
 			(project "pedalsBoard"
-				(path "/423853f6-a5c6-4d97-9a9a-db6f143664c7/26d9f075-73a6-4044-b4f9-8fe225c47fcc/201cb619-540d-483a-b529-2226b2b1f1d1"
-					(reference "C43")
+				(path "/423853f6-a5c6-4d97-9a9a-db6f143664c7/26d9f075-73a6-4044-b4f9-8fe225c47fcc/521dc22e-9478-4c61-a4c9-c65800ada9dd"
+					(reference "C38")
 					(unit 1)
 				)
@@
 		(in_pos_files yes)
 		(dnp no)
-		(property "Reference" "C45"
+		(property "Reference" "C40"
 			(at 189.992 93.98 0)
 			(show_name no)
@@
 		(instances
 			(project "pedalsBoard"
-				(path "/423853f6-a5c6-4d97-9a9a-db6f143664c7/26d9f075-73a6-4044-b4f9-8fe225c47fcc/201cb619-540d-483a-b529-2226b2b1f1d1"
-					(reference "C45")
+				(path "/423853f6-a5c6-4d97-9a9a-db6f143664c7/26d9f075-73a6-4044-b4f9-8fe225c47fcc/521dc22e-9478-4c61-a4c9-c65800ada9dd"
+					(reference "C40")
 					(unit 1)
 				)
@@
 		(in_pos_files yes)
 		(dnp no)
-		(property "Reference" "C42"
+		(property "Reference" "C35"
 			(at 156.718 80.01 0)
 			(show_name no)
@@
 		(instances
 			(project "pedalsBoard"
-				(path "/423853f6-a5c6-4d97-9a9a-db6f143664c7/26d9f075-73a6-4044-b4f9-8fe225c47fcc/201cb619-540d-483a-b529-2226b2b1f1d1"
-					(reference "C42")
+				(path "/423853f6-a5c6-4d97-9a9a-db6f143664c7/26d9f075-73a6-4044-b4f9-8fe225c47fcc/521dc22e-9478-4c61-a4c9-c65800ada9dd"
+					(reference "C35")
 					(unit 1)
 				)
@@
 		(in_pos_files yes)
 		(dnp no)
-		(property "Reference" "#FLG08"
+		(property "Reference" "#FLG010"
 			(at 149.86 84.455 0)
 			(hide yes)
@@
 		(instances
 			(project "pedalsBoard"
-				(path "/423853f6-a5c6-4d97-9a9a-db6f143664c7/26d9f075-73a6-4044-b4f9-8fe225c47fcc/201cb619-540d-483a-b529-2226b2b1f1d1"
-					(reference "#FLG08")
+				(path "/423853f6-a5c6-4d97-9a9a-db6f143664c7/26d9f075-73a6-4044-b4f9-8fe225c47fcc/521dc22e-9478-4c61-a4c9-c65800ada9dd"
+					(reference "#FLG010")
 					(unit 1)
 				)
@@
 		(dnp no)
 		(fields_autoplaced yes)
-		(property "Reference" "R22"
+		(property "Reference" "R32"
 			(at 227.33 85.0899 0)
 			(show_name no)
@@
 		(instances
 			(project "pedalsBoard"
-				(path "/423853f6-a5c6-4d97-9a9a-db6f143664c7/26d9f075-73a6-4044-b4f9-8fe225c47fcc/201cb619-540d-483a-b529-2226b2b1f1d1"
-					(reference "R22")
+				(path "/423853f6-a5c6-4d97-9a9a-db6f143664c7/26d9f075-73a6-4044-b4f9-8fe225c47fcc/521dc22e-9478-4c61-a4c9-c65800ada9dd"
+					(reference "R32")
 					(unit 1)
 				)
@@
 		(dnp no)
 		(fields_autoplaced yes)
-		(property "Reference" "C41"
+		(property "Reference" "C37"
 			(at 105.41 87.6362 0)
 			(show_name no)
@@
 		(instances
 			(project "pedalsBoard"
-				(path "/423853f6-a5c6-4d97-9a9a-db6f143664c7/26d9f075-73a6-4044-b4f9-8fe225c47fcc/201cb619-540d-483a-b529-2226b2b1f1d1"
-					(reference "C41")
+				(path "/423853f6-a5c6-4d97-9a9a-db6f143664c7/26d9f075-73a6-4044-b4f9-8fe225c47fcc/521dc22e-9478-4c61-a4c9-c65800ada9dd"
+					(reference "C37")
 					(unit 1)
 				)
@@
 		(dnp no)
 		(fields_autoplaced yes)
-		(property "Reference" "R23"
+		(property "Reference" "R33"
 			(at 227.33 92.7099 0)
 			(show_name no)
@@
 		(instances
 			(project "pedalsBoard"
-				(path "/423853f6-a5c6-4d97-9a9a-db6f143664c7/26d9f075-73a6-4044-b4f9-8fe225c47fcc/201cb619-540d-483a-b529-2226b2b1f1d1"
-					(reference "R23")
+				(path "/423853f6-a5c6-4d97-9a9a-db6f143664c7/26d9f075-73a6-4044-b4f9-8fe225c47fcc/521dc22e-9478-4c61-a4c9-c65800ada9dd"
+					(reference "R33")
 					(unit 1)
 				)
@@
 		(in_pos_files yes)
 		(dnp no)
-		(property "Reference" "C44"
+		(property "Reference" "C39"
 			(at 173.482 94.234 0)
 			(show_name no)
@@
 		(instances
 			(project "pedalsBoard"
-				(path "/423853f6-a5c6-4d97-9a9a-db6f143664c7/26d9f075-73a6-4044-b4f9-8fe225c47fcc/201cb619-540d-483a-b529-2226b2b1f1d1"
-					(reference "C44")
+				(path "/423853f6-a5c6-4d97-9a9a-db6f143664c7/26d9f075-73a6-4044-b4f9-8fe225c47fcc/521dc22e-9478-4c61-a4c9-c65800ada9dd"
+					(reference "C39")
 					(unit 1)
 				)
@@
 		(instances
 			(project "pedalsBoard"
-				(path "/423853f6-a5c6-4d97-9a9a-db6f143664c7/26d9f075-73a6-4044-b4f9-8fe225c47fcc/201cb619-540d-483a-b529-2226b2b1f1d1"
+				(path "/423853f6-a5c6-4d97-9a9a-db6f143664c7/26d9f075-73a6-4044-b4f9-8fe225c47fcc/521dc22e-9478-4c61-a4c9-c65800ada9dd"
 					(reference "U6")
 					(unit 1)

Commit message: hopefully final before layout
Parts:
- removed TP14: V_in_12V, TestPoint:TestPoint_THTPad_D3.0mm_Drill1.5mm, symbol Connector:TestPoint
- L1: footprint LHRS_Passives:74439369082 -> LHRS_Power:XAL5050822MEC; LCSC P/N (none) -> C5309356; P/N 74439369082 -> XAL5050-822MEC
- R4: renamed from R32; footprint Resistor_SMD:R_0603_1608Metric_Pad0.98x0.95mm_HandSolder -> Resistor_SMD:R_0603_1608Metric
- R6: renamed from R33; footprint Resistor_SMD:R_0603_1608Metric_Pad0.98x0.95mm_HandSolder -> Resistor_SMD:R_0603_1608Metric
- U6: footprint DDC0006A-MFG -> LHRS_ICs:DDC0006A-MFG; LCSC P/N (none) -> C42432812; P/N (none) -> LMR51635XDDCR
- renumbered C36 to C35, C37 to C36, C38 to C37, C39 to C38, C40 to C39, C35 to C4
Other:
- note added: "Vin: 4.6V to 60V"
- note removed: "Test Points"
