File: hardware/VCAT-pedalsBoardPCB/pedalsBoard/USB-C_Connector.kicad_sch (KiCad schematic)
At the start: 6 parts, among them J7 USB_C_Receptacle_USB2.0_16P

Commit message: meow
Parts:
- added C5: 4.7nF, symbol Device:C
- added R4: 1M, symbol Device:R
- renumbered C39 to C55, D8 to D13, D9 to D14, J7 to J9, R20 to R35, R21 to R36
Connections:
- net GND: now also C5.2, R4.2; no longer J9.S1 (SHIELD), J9.S2 (Shield), J9.S3 (Shield), J9.S4 (Shield)
- new net: C5.1, J9.S1 (SHIELD), J9.S2 (Shield), J9.S3 (Shield), J9.S4 (Shield), R4.1

Commit message: test
Parts:
- C5: footprint (none) -> Capacitor_SMD:C_0603_1608Metric_Pad1.08x0.95mm_HandSolder
Changed lines of the file:
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@@
 		(instances
 			(project "pedalsBoard"
-				(path "/423853f6-a5c6-4d97-9a9a-db6f143664c7/09304c86-107a-455a-8167-104f33e31cc1/c7c8ec3c-abef-422a-9eaa-f5640db030e6"
+				(path "/423853f6-a5c6-4d97-9a9a-db6f143664c7/09304c86-107a-455a-8167-104f33e31cc1/533bc9a6-9845-4400-8705-67f71bcf725a"
 					(reference "R35")
 					(unit 1)
@@
 		(instances
 			(project "pedalsBoard"
-				(path "/423853f6-a5c6-4d97-9a9a-db6f143664c7/09304c86-107a-455a-8167-104f33e31cc1/c7c8ec3c-abef-422a-9eaa-f5640db030e6"
+				(path "/423853f6-a5c6-4d97-9a9a-db6f143664c7/09304c86-107a-455a-8167-104f33e31cc1/533bc9a6-9845-4400-8705-67f71bcf725a"
 					(reference "R36")
 					(unit 1)
@@
 			)
 		)
-		(property "Footprint" ""
+		(property "Footprint" "Capacitor_SMD:C_0603_1608Metric_Pad1.08x0.95mm_HandSolder"
 			(at 31.4452 81.28 0)
 			(hide yes)
@@
 		(instances
 			(project "pedalsBoard"
-				(path "/423853f6-a5c6-4d97-9a9a-db6f143664c7/09304c86-107a-455a-8167-104f33e31cc1/c7c8ec3c-abef-422a-9eaa-f5640db030e6"
+				(path "/423853f6-a5c6-4d97-9a9a-db6f143664c7/09304c86-107a-455a-8167-104f33e31cc1/533bc9a6-9845-4400-8705-67f71bcf725a"
 					(reference "C5")
 					(unit 1)
@@
 		(instances
 			(project "pedalsBoard"
-				(path "/423853f6-a5c6-4d97-9a9a-db6f143664c7/09304c86-107a-455a-8167-104f33e31cc1/c7c8ec3c-abef-422a-9eaa-f5640db030e6"
+				(path "/423853f6-a5c6-4d97-9a9a-db6f143664c7/09304c86-107a-455a-8167-104f33e31cc1/533bc9a6-9845-4400-8705-67f71bcf725a"
 					(reference "J9")
 					(unit 1)
@@
 		(instances
 			(project "pedalsBoard"
-				(path "/423853f6-a5c6-4d97-9a9a-db6f143664c7/09304c86-107a-455a-8167-104f33e31cc1/c7c8ec3c-abef-422a-9eaa-f5640db030e6"
+				(path "/423853f6-a5c6-4d97-9a9a-db6f143664c7/09304c86-107a-455a-8167-104f33e31cc1/533bc9a6-9845-4400-8705-67f71bcf725a"
 					(reference "#FLG010")
 					(unit 1)
@@
 		(instances
 			(project "pedalsBoard"
-				(path "/423853f6-a5c6-4d97-9a9a-db6f143664c7/09304c86-107a-455a-8167-104f33e31cc1/c7c8ec3c-abef-422a-9eaa-f5640db030e6"
+				(path "/423853f6-a5c6-4d97-9a9a-db6f143664c7/09304c86-107a-455a-8167-104f33e31cc1/533bc9a6-9845-4400-8705-67f71bcf725a"
 					(reference "D13")
 					(unit 1)
@@
 		(instances
 			(project "pedalsBoard"
-				(path "/423853f6-a5c6-4d97-9a9a-db6f143664c7/09304c86-107a-455a-8167-104f33e31cc1/c7c8ec3c-abef-422a-9eaa-f5640db030e6"
+				(path "/423853f6-a5c6-4d97-9a9a-db6f143664c7/09304c86-107a-455a-8167-104f33e31cc1/533bc9a6-9845-4400-8705-67f71bcf725a"
 					(reference "R4")
 					(unit 1)
@@
 		(instances
 			(project "pedalsBoard"
-				(path "/423853f6-a5c6-4d97-9a9a-db6f143664c7/09304c86-107a-455a-8167-104f33e31cc1/c7c8ec3c-abef-422a-9eaa-f5640db030e6"
+				(path "/423853f6-a5c6-4d97-9a9a-db6f143664c7/09304c86-107a-455a-8167-104f33e31cc1/533bc9a6-9845-4400-8705-67f71bcf725a"
 					(reference "C55")
 					(unit 1)
@@
 		(instances
 			(project "pedalsBoard"
-				(path "/423853f6-a5c6-4d97-9a9a-db6f143664c7/09304c86-107a-455a-8167-104f33e31cc1/c7c8ec3c-abef-422a-9eaa-f5640db030e6"
+				(path "/423853f6-a5c6-4d97-9a9a-db6f143664c7/09304c86-107a-455a-8167-104f33e31cc1/533bc9a6-9845-4400-8705-67f71bcf725a"
 					(reference "D14")
 					(unit 1)

Commit message: addressed review, brake switch on slack
Parts:
- renumbered C55 to C3, C5 to C4, D13 to D2, D14 to D3, J9 to J6, R35 to R2, R36 to R3
Changed lines of the file:
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@@
 		(in_pos_files yes)
 		(dnp no)
-		(property "Reference" "R35"
+		(property "Reference" "R2"
 			(at 86.106 48.26 90)
 			(show_name no)
@@
 		(instances
 			(project "pedalsBoard"
-				(path "/423853f6-a5c6-4d97-9a9a-db6f143664c7/09304c86-107a-455a-8167-104f33e31cc1/533bc9a6-9845-4400-8705-67f71bcf725a"
-					(reference "R35")
+				(path "/423853f6-a5c6-4d97-9a9a-db6f143664c7/09304c86-107a-455a-8167-104f33e31cc1/d1a0b1bd-dedf-4da6-ad23-b1fcccb3d646"
+					(reference "R2")
 					(unit 1)
 				)
@@
 		(in_pos_files yes)
 		(dnp no)
-		(property "Reference" "R36"
+		(property "Reference" "R3"
 			(at 93.726 48.26 90)
 			(show_name no)
@@
 		(instances
 			(project "pedalsBoard"
-				(path "/423853f6-a5c6-4d97-9a9a-db6f143664c7/09304c86-107a-455a-8167-104f33e31cc1/533bc9a6-9845-4400-8705-67f71bcf725a"
-					(reference "R36")
+				(path "/423853f6-a5c6-4d97-9a9a-db6f143664c7/09304c86-107a-455a-8167-104f33e31cc1/d1a0b1bd-dedf-4da6-ad23-b1fcccb3d646"
+					(reference "R3")
 					(unit 1)
 				)
@@
 		(in_pos_files yes)
 		(dnp no)
-		(property "Reference" "C5"
+		(property "Reference" "C4"
 			(at 31.75 73.152 0)
 			(show_name no)
@@
 		(instances
 			(project "pedalsBoard"
-				(path "/423853f6-a5c6-4d97-9a9a-db6f143664c7/09304c86-107a-455a-8167-104f33e31cc1/533bc9a6-9845-4400-8705-67f71bcf725a"
-					(reference "C5")
+				(path "/423853f6-a5c6-4d97-9a9a-db6f143664c7/09304c86-107a-455a-8167-104f33e31cc1/d1a0b1bd-dedf-4da6-ad23-b1fcccb3d646"
+					(reference "C4")
 					(unit 1)
 				)
@@
 		(dnp no)
 		(fields_autoplaced yes)
-		(property "Reference" "J9"
+		(property "Reference" "J6"
 			(at 35.56 22.86 0)
 			(show_name no)
@@
 		(instances
 			(project "pedalsBoard"
-				(path "/423853f6-a5c6-4d97-9a9a-db6f143664c7/09304c86-107a-455a-8167-104f33e31cc1/533bc9a6-9845-4400-8705-67f71bcf725a"
-					(reference "J9")
+				(path "/423853f6-a5c6-4d97-9a9a-db6f143664c7/09304c86-107a-455a-8167-104f33e31cc1/d1a0b1bd-dedf-4da6-ad23-b1fcccb3d646"
+					(reference "J6")
 					(unit 1)
 				)
@@
 		(dnp no)
 		(fields_autoplaced yes)
-		(property "Reference" "#FLG010"
+		(property "Reference" "#FLG07"
 			(at 71.755 30.48 0)
 			(hide yes)
@@
 		(instances
 			(project "pedalsBoard"
-				(path "/423853f6-a5c6-4d97-9a9a-db6f143664c7/09304c86-107a-455a-8167-104f33e31cc1/533bc9a6-9845-4400-8705-67f71bcf725a"
-					(reference "#FLG010")
+				(path "/423853f6-a5c6-4d97-9a9a-db6f143664c7/09304c86-107a-455a-8167-104f33e31cc1/d1a0b1bd-dedf-4da6-ad23-b1fcccb3d646"
+					(reference "#FLG07")
 					(unit 1)
 				)
@@
 		(in_pos_files yes)
 		(dnp no)
-		(property "Reference" "D13"
+		(property "Reference" "D2"
 			(at 59.69 24.765 0)
 			(show_name no)
@@
 		(instances
 			(project "pedalsBoard"
-				(path "/423853f6-a5c6-4d97-9a9a-db6f143664c7/09304c86-107a-455a-8167-104f33e31cc1/533bc9a6-9845-4400-8705-67f71bcf725a"
-					(reference "D13")
+				(path "/423853f6-a5c6-4d97-9a9a-db6f143664c7/09304c86-107a-455a-8167-104f33e31cc1/d1a0b1bd-dedf-4da6-ad23-b1fcccb3d646"
+					(reference "D2")
 					(unit 1)
 				)
@@
 		(instances
 			(project "pedalsBoard"
-				(path "/423853f6-a5c6-4d97-9a9a-db6f143664c7/09304c86-107a-455a-8167-104f33e31cc1/533bc9a6-9845-4400-8705-67f71bcf725a"
+				(path "/423853f6-a5c6-4d97-9a9a-db6f143664c7/09304c86-107a-455a-8167-104f33e31cc1/d1a0b1bd-dedf-4da6-ad23-b1fcccb3d646"
 					(reference "R4")
 					(unit 1)
@@
 		(in_pos_files yes)
 		(dnp no)
-		(property "Reference" "C55"
+		(property "Reference" "C3"
 			(at 64.3128 37.9984 0)
 			(show_name no)
@@
 		(instances
 			(project "pedalsBoard"
-				(path "/423853f6-a5c6-4d97-9a9a-db6f143664c7/09304c86-107a-455a-8167-104f33e31cc1/533bc9a6-9845-4400-8705-67f71bcf725a"
-					(reference "C55")
+				(path "/423853f6-a5c6-4d97-9a9a-db6f143664c7/09304c86-107a-455a-8167-104f33e31cc1/d1a0b1bd-dedf-4da6-ad23-b1fcccb3d646"
+					(reference "C3")
 					(unit 1)
 				)
@@
 		(in_pos_files yes)
 		(dnp no)
-		(property "Reference" "D14"
+		(property "Reference" "D3"
 			(at 82.55 71.12 0)
 			(show_name no)
@@
 		(instances
 			(project "pedalsBoard"
-				(path "/423853f6-a5c6-4d97-9a9a-db6f143664c7/09304c86-107a-455a-8167-104f33e31cc1/533bc9a6-9845-4400-8705-67f71bcf725a"
-					(reference "D14")
+				(path "/423853f6-a5c6-4d97-9a9a-db6f143664c7/09304c86-107a-455a-8167-104f33e31cc1/d1a0b1bd-dedf-4da6-ad23-b1fcccb3d646"
+					(reference "D3")
 					(unit 1)
 				)

Commit message: hopefully final before layout
Parts:
- removed C4: 4.7nF, Capacitor_SMD:C_0603_1608Metric_Pad1.08x0.95mm_HandSolder, symbol Device:C
- removed D3: TPD2EUSB30DRTR, LHRS_ICs:TPD2EUSB30DRTR, symbol lhrs_ics:TPD2EUSB30DRTR
- removed R4: 1M, symbol Device:R
- added D3: SP0503BAHT, Package_TO_SOT_SMD:SOT-143, symbol lhrs_ics:SP0503BAH
- C3: value 10uF -> 10u
- J1: renamed from J6; footprint LHRS_ICs:USB_C_Receptacle_GCT_USB4105-xx-A_16P_TopMnt_Horizontal -> LHRS_Connectors:USB_C_Receptacle_GCT_USB4105-xx-A_16P_TopMnt_Horizontal
Connections:
- net GND: now also J1.S1 (SHIELD), J1.S2 (Shield), J1.S3 (Shield), J1.S4 (Shield), D3.1 (A)
- net VBUS_IN: now also D3.4 (K)
- net USB_DM renamed USB_D-
- net USB_D-: now also D3.3 (K)
- net USB_DP renamed USB_D+
- net USB_D+: now also D3.2 (K)
Other:
- note removed: "5.5V working 7V breakdown 8V clamping"
