File: hardware/VCAT-pedalsBoardPCB/pedalsBoard/CAN_Transceiver.kicad_sch (KiCad schematic)
At the start: 9 parts, among them IC1 TCAN3413DR

Commit message: test
Connections:
- net 3.3v renamed 3.3V
Changed lines of the file:
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@@
 		)
 	)
-	(hierarchical_label "3.3v"
+	(hierarchical_label "3.3V"
 		(shape input)
 		(at 149.86 67.31 0)
@@
 		)
 	)
-	(hierarchical_label "3.3v"
+	(hierarchical_label "3.3V"
 		(shape input)
 		(at 87.63 63.5 0)

Commit message: addressed review, brake switch on slack
Parts:
- renumbered C16 to C27, C17 to C28, C18 to C29, C19 to C30, D4 to D13, JP1 to JP2, R9 to R29, R10 to R30
Changed lines of the file:
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@@
 		(in_pos_files yes)
 		(dnp no)
-		(property "Reference" "C17"
+		(property "Reference" "C28"
 			(at 76.2 73.66 0)
 			(show_name no)
@@
 		(instances
 			(project "pedalsBoard"
-				(path "/423853f6-a5c6-4d97-9a9a-db6f143664c7/aafb20a0-2a2f-4620-a8da-8fa8b138f682"
-					(reference "C17")
+				(path "/423853f6-a5c6-4d97-9a9a-db6f143664c7/30d55949-b7b9-413e-9bcf-a768f52b2f03"
+					(reference "C28")
 					(unit 1)
 				)
@@
 		(in_pos_files yes)
 		(dnp no)
-		(property "Reference" "C19"
+		(property "Reference" "C30"
 			(at 194.564 88.646 0)
 			(show_name no)
@@
 		(instances
 			(project "pedalsBoard"
-				(path "/423853f6-a5c6-4d97-9a9a-db6f143664c7/aafb20a0-2a2f-4620-a8da-8fa8b138f682"
-					(reference "C19")
+				(path "/423853f6-a5c6-4d97-9a9a-db6f143664c7/30d55949-b7b9-413e-9bcf-a768f52b2f03"
+					(reference "C30")
 					(unit 1)
 				)
@@
 		(dnp no)
 		(fields_autoplaced yes)
-		(property "Reference" "JP1"
+		(property "Reference" "JP2"
 			(at 215.9 78.74 0)
 			(show_name no)
@@
 		(instances
 			(project "pedalsBoard"
-				(path "/423853f6-a5c6-4d97-9a9a-db6f143664c7/aafb20a0-2a2f-4620-a8da-8fa8b138f682"
-					(reference "JP1")
+				(path "/423853f6-a5c6-4d97-9a9a-db6f143664c7/30d55949-b7b9-413e-9bcf-a768f52b2f03"
+					(reference "JP2")
 					(unit 1)
 				)
@@
 		(in_pos_files yes)
 		(dnp no)
-		(property "Reference" "C18"
+		(property "Reference" "C29"
 			(at 88.138 73.66 0)
 			(show_name no)
@@
 		(instances
 			(project "pedalsBoard"
-				(path "/423853f6-a5c6-4d97-9a9a-db6f143664c7/aafb20a0-2a2f-4620-a8da-8fa8b138f682"
-					(reference "C18")
+				(path "/423853f6-a5c6-4d97-9a9a-db6f143664c7/30d55949-b7b9-413e-9bcf-a768f52b2f03"
+					(reference "C29")
 					(unit 1)
 				)
@@
 		(in_pos_files yes)
 		(dnp no)
-		(property "Reference" "C16"
+		(property "Reference" "C27"
 			(at 65.278 73.66 0)
 			(show_name no)
@@
 		(instances
 			(project "pedalsBoard"
-				(path "/423853f6-a5c6-4d97-9a9a-db6f143664c7/aafb20a0-2a2f-4620-a8da-8fa8b138f682"
-					(reference "C16")
+				(path "/423853f6-a5c6-4d97-9a9a-db6f143664c7/30d55949-b7b9-413e-9bcf-a768f52b2f03"
+					(reference "C27")
 					(unit 1)
 				)
@@
 		(in_pos_files yes)
 		(dnp no)
-		(property "Reference" "R10"
+		(property "Reference" "R30"
 			(at 201.93 80.01 90)
 			(show_name no)
@@
 		(instances
 			(project "pedalsBoard"
-				(path "/423853f6-a5c6-4d97-9a9a-db6f143664c7/aafb20a0-2a2f-4620-a8da-8fa8b138f682"
-					(reference "R10")
+				(path "/423853f6-a5c6-4d97-9a9a-db6f143664c7/30d55949-b7b9-413e-9bcf-a768f52b2f03"
+					(reference "R30")
 					(unit 1)
 				)
@@
 		(dnp no)
 		(fields_autoplaced yes)
-		(property "Reference" "D4"
+		(property "Reference" "D13"
 			(at 196.85 46.99 0)
 			(show_name no)
@@
 		(instances
 			(project "pedalsBoard"
-				(path "/423853f6-a5c6-4d97-9a9a-db6f143664c7/aafb20a0-2a2f-4620-a8da-8fa8b138f682"
-					(reference "D4")
+				(path "/423853f6-a5c6-4d97-9a9a-db6f143664c7/30d55949-b7b9-413e-9bcf-a768f52b2f03"
+					(reference "D13")
 					(unit 1)
 				)
@@
 		(instances
 			(project "pedalsBoard"
-				(path "/423853f6-a5c6-4d97-9a9a-db6f143664c7/aafb20a0-2a2f-4620-a8da-8fa8b138f682"
+				(path "/423853f6-a5c6-4d97-9a9a-db6f143664c7/30d55949-b7b9-413e-9bcf-a768f52b2f03"
 					(reference "IC1")
 					(unit 1)
@@
 		(in_pos_files yes)
 		(dnp no)
-		(property "Reference" "R9"
+		(property "Reference" "R29"
 			(at 176.53 80.01 90)
 			(show_name no)
@@
 		(instances
 			(project "pedalsBoard"
-				(path "/423853f6-a5c6-4d97-9a9a-db6f143664c7/aafb20a0-2a2f-4620-a8da-8fa8b138f682"
-					(reference "R9")
-					(unit 1)
-				)
+				(path "/423853f6-a5c6-4d97-9a9a-db6f143664c7/30d55949-b7b9-413e-9bcf-a768f52b2f03"
+					(reference "R29")
+					(unit 1)
+				)
